File: dev-kit/Power.kicad_sch (KiCad schematic)
At the start: 26 parts, among them IC101 nPM1300-QEXX, X101 Battery, X102 Battery, X103 Power

Commit message: Bug: Issue #121
Signed-off-by: Daniel Kampert <DanielKampert@kampis-elektroecke.de>
Parts:
- X103: manf# 10129380-904002ALF -> 77311-818-02LF
Connections:
- net GND: now also X101.2 (Pin_2); no longer X101.1 (Pin_1)
- net VBAT: now also X101.1 (Pin_1); no longer X101.2 (Pin_2)
Changed lines of the file:
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@@
 			)
 		)
-		(property "Datasheet" "https://cdn.amphenol-cs.com/media/wysiwyg/files/documentation/datasheet/boardwiretoboard/bwb_econostik_254headers.pdf"
+		(property "Datasheet" "https://www.mouser.de/datasheet/2/18/2/bwb_bergstik-3370040.pdf"
 			(at 275.59 151.13 0)
 			(effects
@@
 			)
 		)
-		(property "manf#" "10129380-904002ALF"
+		(property "manf#" "77311-818-02LF"
 			(at 275.59 151.13 0)
 			(effects
@@
 	(symbol
 		(lib_id "Connector_Generic:Conn_01x02")
-		(at 160.02 30.48 0)
+		(at 160.02 33.02 0)
+		(mirror x)
 		(unit 1)
 		(exclude_from_sim no)
@@
 		(fields_autoplaced yes)
 		(property "Reference" "X101"
-			(at 162.56 30.4799 0)
-			(effects
-				(font
-					(size 1.27 1.27)
-				)
-				(justify left)
+			(at 160.02 24.13 0)
+			(effects
+				(font
+					(size 1.27 1.27)
+				)
 			)
 		)
 		(property "Value" "Battery"
-			(at 162.56 33.0199 0)
-			(effects
-				(font
-					(size 1.27 1.27)
-				)
-				(justify left)
+			(at 160.02 26.67 0)
+			(effects
+				(font
+					(size 1.27 1.27)
+				)
 			)
 		)
 		(property "Footprint" "Connector_PinHeader_2.54mm:PinHeader_1x02_P2.54mm_Vertical"
-			(at 160.02 30.48 0)
+			(at 160.02 33.02 0)
 			(effects
 				(font
@@
 		)
 		(property "Datasheet" "https://cdn.amphenol-cs.com/media/wysiwyg/files/documentation/datasheet/boardwiretoboard/bwb_econostik_254headers.pdf"
-			(at 160.02 30.48 0)
+			(at 160.02 33.02 0)
 			(effects
 				(font
@@
 		)
 		(property "Description" "Generic connector, single row, 01x02, script generated (kicad-library-utils/schlib/autogen/connector/)"
-			(at 160.02 30.48 0)
+			(at 160.02 33.02 0)
 			(effects
 				(font
@@
 		)
 		(property "manf" "Amphenol FCI"
-			(at 160.02 30.48 0)
+			(at 160.02 33.02 0)
 			(effects
 				(font
@@
 		)
 		(property "manf#" "10129380-902001BLF"
-			(at 160.02 30.48 0)
+			(at 160.02 33.02 0)
 			(effects
 				(font
@@
 		)
 		(property "mouser#" "649-1012938090201BLF"
-			(at 160.02 30.48 0)
+			(at 160.02 33.02 0)
 			(effects
 				(font
@@
 		)
 		(property "CONFIG" ""
-			(at 160.02 30.48 0)
-			(effects
-				(font
+			(at 160.02 33.02 0)
+			(effects
+				(font
