File: devkit/Power.kicad_sch (KiCad schematic)
At the start: 40 parts, among them IC401 nPM1300-QEXX, Q401 PMZ550UNEYL, Q402 PMZ550UNEYL, Q403 PMZ550UNEYL, Q404 PMZB320UPEYL, X401 Battery, X402 Battery, X403 Power

Commit message: Bug: Issue #158
- Fix silkscreens
- Add pull-up resistors to I2C lines
- Set the Pull-Up for Flash CS to NA
- Fix wrong part number for the I2C header

Closes #158

Signed-off-by: Daniel Kampert <DanielKampert@kampis-elektroecke.de>
Parts:
- renumbered C410 to C404, C404 to C405, C405 to C406, C406 to C407, C407 to C408, C408 to C409, C409 to C410, TP405 to TP403, TP403 to TP404, TP404 to TP405
