File: devkit/Peripherals.kicad_sch (KiCad schematic)
At the start: 50 parts, among them IC501 APDS-9306-065, IC502 BMI270, IC503 LIS2MDLTR, IC504 BMP581, IC505 DRV2603RUNT, IC506 PCA9306JK, IC507 RV-8263-C8, J501 Jumper, J502 Jumper, J503 Jumper, J504 Jumper, J505 Jumper, J506 Jumper, J507 Jumper, M501 Vibrator DC Motor, X501 Current, X502 I2S, X503 Current, X504 I2C, X505 Current, X506 Current, X507 Current, X508 Current, X509 Motor, X510 Current

Commit message: Changes
Parts:
- IC502: value BMI270 -> ThisIsAWrongValue
Changed lines of the file:
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@@
 			)
 		)
-		(property "Value" "BMI270"
+		(property "Value" "ThisIsAWrongValue"
 			(at 185.42 92.71 0)
 			(effects
